File: Microcontroller.kicad_sch (KiCad schematic)
At the start: 10 parts, among them U7 ESP32-S3-WROOM-1

Commit message: Round board corners, re-annotate test points, rewrite README for GitHub
Board: 1.0 mm radius corners; outline now 71.00 x 46.00 mm.
Schematic: test points re-annotated to signal names (SDA1, SLC1,
CSN1, CLK1, MOSI1, MISO1, VS1, G1, G2, IO7, IO15, IO47, RST1, BOOT1).

README rewritten as a GitHub landing page: explains what the board is
for, adds Mermaid system-architecture and power-path diagrams, a
verified pin map traced from the netlist, board specs, and fab
instructions. Drops the ERC/DRC status and issue-tracking sections.

Co-Authored-By: Claude Opus 5 <noreply@anthropic.com>
Parts:
- renumbered JP2 to BOOT1, JP1 to RST1
Connections:
- net IO47: now reaches U7.24 (IO47)
Changed lines of the file:
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@@
+		)
+	)
+	(hierarchical_label "IO47"
+		(shape bidirectional)
+		(at 140.97 92.71 0)
+		(effects
+			(font
+				(size 1.27 1.27)
+			)
+			(justify left)
 		)
 	)
@@
 		(dnp no)
 		(fields_autoplaced yes)
-		(property "Reference" "JP1"
+		(property "Reference" "RST1"
 			(at 184.15 77.4699 90)
 			(show_name no)
@@
 			(project "meshtastic-v0"
 				(path "/e4d6fcd6-7415-4955-88fd-f0e430797514/b95685e3-53f8-4d4b-b7ad-2a266b169b28"
-					(reference "JP1")
+					(reference "RST1")
 					(unit 1)
 				)
@@
 		(dnp no)
 		(fields_autoplaced yes)
-		(property "Reference" "JP2"
+		(property "Reference" "BOOT1"
 			(at 172.72 77.4699 90)
 			(show_name no)
@@
 			(project "meshtastic-v0"
 				(path "/e4d6fcd6-7415-4955-88fd-f0e430797514/b95685e3-53f8-4d4b-b7ad-2a266b169b28"
-					(reference "JP2")
+					(reference "BOOT1")
 					(unit 1)
 				)
