File: Microcontroller.kicad_sch (KiCad schematic)
At the start: 10 parts, among them U7 ESP32-S3-WROOM-1

Commit message: vib motor
Connections:
- net IO7 renamed VIB_MTR
Changed lines of the file:
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@@
+		)
+	)
+	(hierarchical_label "VIB_MTR"
+		(shape output)
+		(at 105.41 72.39 180)
+		(effects
+			(font
+				(size 1.27 1.27)
+			)
+			(justify right)
 		)
 	)
@@
 		(effects
 			(font
-				(size 1.27 1.27)
-			)
-			(justify right)
-		)
-	)
-	(hierarchical_label "IO7"
-		(shape bidirectional)
-		(at 105.41 72.39 180)
-		(effects
-			(font

Commit message: added vib motor fix
Connections:
- net IO15 is gone; now on net VIB_MTR: U7.8 (IO15)
- net VIB_MTR: no longer U7.7 (IO7)
- new net IO07: U7.7 (IO7)
Changed lines of the file:
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@@
+		)
+	)
+	(hierarchical_label "VIB_MTR"
+		(shape output)
+		(at 105.41 92.71 180)
+		(effects
+			(font
+				(size 1.27 1.27)
+			)
+			(justify right)
 		)
 	)
@@
 		)
 	)
-	(hierarchical_label "VIB_MTR"
-		(shape output)
+	(hierarchical_label "IO07"
+		(shape bidirectional)
 		(at 105.41 72.39 180)
 		(effects
@@
 		)
 	)
-	(hierarchical_label "IO15"
-		(shape bidirectional)
-		(at 105.41 92.71 180)
-		(effects
-			(font
-				(size 1.27 1.27)
-			)
-			(justify right)
-		)
-	)
