File: Peripherals.kicad_sch (KiCad schematic)
At the start: 18 parts, among them Q1 SI2302

Commit message: Round board corners, re-annotate test points, rewrite README for GitHub
Board: 1.0 mm radius corners; outline now 71.00 x 46.00 mm.
Schematic: test points re-annotated to signal names (SDA1, SLC1,
CSN1, CLK1, MOSI1, MISO1, VS1, G1, G2, IO7, IO15, IO47, RST1, BOOT1).

README rewritten as a GitHub landing page: explains what the board is
for, adds Mermaid system-architecture and power-path diagrams, a
verified pin map traced from the netlist, board specs, and fab
instructions. Drops the ERC/DRC status and issue-tracking sections.

Co-Authored-By: Claude Opus 5 <noreply@anthropic.com>
Parts:
- added IO47: IO47, TestPoint:TestPoint_Pad_1.0x1.0mm, symbol Connector:TestPoint
- renumbered TP22 to 3V3, TP15 to CLK1, TP14 to CSN1, TP23 to G1, TP26 to G2, TP19 to IO15, TP18 to IO7, TP17 to MISO1, TP16 to MOSI1, TP12 to SDA1, TP13 to SLC1, TP21 to VS1
Connections:
- new net IO47: IO47.1
Changed lines of the file:
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@@
+	(wire
+		(pts
+			(xy 129.54 102.87) (xy 133.35 102.87)
+		)
+		(stroke
+			(width 0)
+			(type default)
+		)
+	)
 	(wire
 		(pts
@@
 		(pts
 			(xy 172.72 72.39) (xy 172.72 77.47)
+		)
+		(stroke
+			(width 0)
+			(type default)
+		)
+	)
+	(wire
+		(pts
+			(xy 133.35 102.87) (xy 133.35 109.22)
+		)
+		(stroke
+			(width 0)
+			(type default)
+		)
+	)
+	(wire
+		(pts
+			(xy 133.35 109.22) (xy 138.43 109.22)
 		)
 		(stroke
@@
 		(shape input)
 		(at 132.08 128.27 180)
+		(effects
+			(font
+				(size 1.27 1.27)
+			)
+			(justify right)
+		)
+	)
+	(hierarchical_label "IO47"
+		(shape bidirectional)
+		(at 129.54 102.87 180)
 		(effects
 			(font
@@
 		(dnp no)
 		(fields_autoplaced yes)
-		(property "Reference" "TP12"
+		(property "Reference" "SDA1"
 			(at 102.87 102.8699 90)
 			(show_name no)
@@
 			(project "meshtastic-v0"
 				(path "/e4d6fcd6-7415-4955-88fd-f0e430797514/159c1940-45ee-4eb6-b2c7-3caab0dbb038"
-					(reference "TP12")
+					(reference "SDA1")
 					(unit 1)
 				)
@@
 		(dnp no)
 		(fields_autoplaced yes)
-		(property "Reference" "TP21"
+		(property "Reference" "VS1"
 			(at 95.25 121.9199 90)
 			(show_name no)
@@
 			(project "meshtastic-v0"
 				(path "/e4d6fcd6-7415-4955-88fd-f0e430797514/159c1940-45ee-4eb6-b2c7-3caab0dbb038"
-					(reference "TP21")
+					(reference "VS1")
 					(unit 1)
 				)
@@
 		(dnp no)
 		(fields_autoplaced yes)
-		(property "Reference" "TP17"
+		(property "Reference" "MISO1"
 			(at 149.86 142.2399 90)
 			(show_name no)
@@
 			(project "meshtastic-v0"
 				(path "/e4d6fcd6-7415-4955-88fd-f0e430797514/159c1940-45ee-4eb6-b2c7-3caab0dbb038"
-					(reference "TP17")
+					(reference "MISO1")
 					(unit 1)
 				)
@@
 		(dnp no)
 		(fields_autoplaced yes)
-		(property "Reference" "TP15"
+		(property "Reference" "CLK1"
 			(at 149.86 132.0799 90)
 			(show_name no)
@@
 			(project "meshtastic-v0"
 				(path "/e4d6fcd6-7415-4955-88fd-f0e430797514/159c1940-45ee-4eb6-b2c7-3caab0dbb038"
-					(reference "TP15")
+					(reference "CLK1")
 					(unit 1)
 				)
@@
 		(dnp no)
 		(fields_autoplaced yes)
-		(property "Reference" "TP26"
+		(property "Reference" "G2"
 			(at 95.25 137.1599 90)
 			(show_name no)
@@
 			(project "meshtastic-v0"
 				(path "/e4d6fcd6-7415-4955-88fd-f0e430797514/159c1940-45ee-4eb6-b2c7-3caab0dbb038"
-					(reference "TP26")
+					(reference "G2")
 					(unit 1)
 				)
@@
 		(dnp no)
 		(fields_autoplaced yes)
-		(property "Reference" "TP23"
+		(property "Reference" "G1"
 			(at 95.25 132.0799 90)
 			(show_name no)
@@
 			(project "meshtastic-v0"
 				(path "/e4d6fcd6-7415-4955-88fd-f0e430797514/159c1940-45ee-4eb6-b2c7-3caab0dbb038"
-					(reference "TP23")
+					(reference "G1")
 					(unit 1)
 				)
@@
 		(dnp no)
 		(fields_autoplaced yes)
-		(property "Reference" "TP14"
+		(property "Reference" "CSN1"
 			(at 149.86 126.9999 90)
 			(show_name no)
@@
 			(project "meshtastic-v0"
 				(path "/e4d6fcd6-7415-4955-88fd-f0e430797514/159c1940-45ee-4eb6-b2c7-3caab0dbb038"
-					(reference "TP14")
+					(reference "CSN1")
 					(unit 1)
 				)
@@
 		(dnp no)
 		(fields_autoplaced yes)
-		(property "Reference" "TP13"
+		(property "Reference" "SLC1"
 			(at 102.87 107.9499 90)
 			(show_name no)
@@
 			(project "meshtastic-v0"
 				(path "/e4d6fcd6-7415-4955-88fd-f0e430797514/159c1940-45ee-4eb6-b2c7-3caab0dbb038"
-					(reference "TP13")
+					(reference "SLC1")
 					(unit 1)
 				)
@@
 		(dnp no)
 		(fields_autoplaced yes)
-		(property "Reference" "TP16"
+		(property "Reference" "MOSI1"
 			(at 149.86 137.1599 90)
 			(show_name no)
@@
 			(project "meshtastic-v0"
 				(path "/e4d6fcd6-7415-4955-88fd-f0e430797514/159c1940-45ee-4eb6-b2c7-3caab0dbb038"
-					(reference "TP16")
+					(reference "MOSI1")
 					(unit 1)
 				)
@@
 		(dnp no)
 		(fields_autoplaced yes)
-		(property "Reference" "TP19"
+		(property "Reference" "IO15"
 			(at 143.51 101.5999 90)
 			(show_name no)
@@
 			(project "meshtastic-v0"
 				(path "/e4d6fcd6-7415-4955-88fd-f0e430797514/159c1940-45ee-4eb6-b2c7-3caab0dbb038"
-					(reference "TP19")
+					(reference "IO15")
 					(unit 1)
 				)
@@
 		(dnp no)
 		(fields_autoplaced yes)
-		(property "Reference" "TP22"
+		(property "Reference" "3V3"
 			(at 95.25 126.9999 90)
 			(show_name no)
@@
 			(project "meshtastic-v0"
 				(path "/e4d6fcd6-7415-4955-88fd-f0e430797514/159c1940-45ee-4eb6-b2c7-3caab0dbb038"
-					(reference "TP22")
+					(reference "3V3")
 					(unit 1)
 				)
@@
 		(dnp no)
 		(fields_autoplaced yes)
-		(property "Reference" "TP18"
+		(property "Reference" "IO7"
 			(at 143.51 96.5199 90)
 			(show_name no)
@@
 			(project "meshtastic-v0"
 				(path "/e4d6fcd6-7415-4955-88fd-f0e430797514/159c1940-45ee-4eb6-b2c7-3caab0dbb038"
-					(reference "TP18")
+					(reference "IO7")
 					(unit 1)
 				)
+			)
+		)
+	)
+	(symbol
+		(lib_id "Connector:TestPoint")
+		(at 138.43 109.22 270)
+		(unit 1)
+		(body_style 1)
+		(exclude_from_sim no)
+		(in_bom yes)
+		(on_board yes)
+		(in_pos_files yes)
+		(dnp no)
+		(fields_autoplaced yes)
+		(property "Reference" "IO47"
+			(at 143.51 107.9499 90)
+			(show_name no)
+			(do_not_autoplace no)
+			(effects
+				(font
+					(size 1.27 1.27)
+				)
+				(justify left)
+			)
+		)
+		(property "Value" "IO47"
+			(at 143.51 110.4899 90)
+			(show_name no)
+			(do_not_autoplace no)
+			(effects
+				(font
+					(size 1.27 1.27)
+				)
+				(justify left)
+			)
+		)
+		(property "Footprint" "TestPoint:TestPoint_Pad_1.0x1.0mm"
+			(at 138.43 114.3 0)
+			(hide yes)
+			(show_name no)
+			(do_not_autoplace no)
+			(effects
+				(font
+					(size 1.27 1.27)
+				)
+			)
+		)
+		(property "Datasheet" ""
+			(at 138.43 114.3 0)
+			(hide yes)
+			(show_name no)
+			(do_not_autoplace no)
+			(effects
+				(font
+					(size 1.27 1.27)
+				)
+			)
+		)
+		(property "Description" "test point"
+			(at 138.43 109.22 0)
+			(hide yes)
+			(show_name no)
+			(do_not_autoplace no)
+			(effects
+				(font
+					(size 1.27 1.27)
+				)
+			)
+		)
+		(pin "1"
+		)
+		(instances
+			(project "meshtastic-v0"
+				(path "/e4d6fcd6-7415-4955-88fd-f0e430797514/159c1940-45ee-4eb6-b2c7-3caab0dbb038"
+					(reference "IO47")
+					(unit 1)
+				)
