File: Peripherals.kicad_sch (KiCad schematic)
At the start: 19 parts, among them Q1 SI2302

Commit message: vib motor
Parts:
- removed IO7: IO7, TestPoint:TestPoint_Pad_1.0x1.0mm, symbol Connector:TestPoint
- added D9: 1N5819WS, Diode_SMD:D_SOD-323, symbol Diode:1N5819WS
- added JP1: SolderJumper_2_Open, Jumper:SolderJumper-2_P1.3mm_Open_Pad1.0x1.5mm, symbol Jumper:SolderJumper_2_Open
- added Q4: SI2302, Package_TO_SOT_SMD:SOT-23, symbol Transistor_FET:DMN2040U
- added R23: 10k, Resistor_SMD:R_0805_2012Metric, symbol Device:R
Connections:
- net +3V3: now also D9.1 (K), JP1.2 (B)
- net GND: now also Q4.2 (S), R23.1
- new net: D9.2 (A), JP1.1 (A), Q4.3 (D)
- new net VIB_MTR: Q4.1 (G), R23.2

Commit message: added vib motor fix
Parts:
- renumbered IO15 to IO07
Connections:
- net IO15 renamed IO07
Changed lines of the file:
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@@
 		)
 	)
-	(hierarchical_label "IO15"
+	(hierarchical_label "IO07"
 		(shape bidirectional)
 		(at 129.54 100.33 180)
@@
 		(dnp no)
 		(fields_autoplaced yes)
-		(property "Reference" "IO15"
+		(property "Reference" "IO07"
 			(at 143.51 101.5999 90)
 			(show_name no)
@@
 			(project "meshtastic-v0"
 				(path "/e4d6fcd6-7415-4955-88fd-f0e430797514/159c1940-45ee-4eb6-b2c7-3caab0dbb038"
-					(reference "IO15")
-					(unit 1)
-				)
+					(reference "IO07")
+					(unit 1)
+				)
