File: meshtastic-v0.kicad_pcb (KiCad board)
At the start: 2 copper layers, 71 x 46.1 mm, 87 parts, among them J1 USB_C_Receptacle_USB2.0_16P, J2 Conn_01x02_Pin, J3 Conn_Coaxial, J4 Conn_Coaxial, Q1 SI2302, Q2 Q_PNP_BEC, Q3 Q_NPN_BEC, U1 DM-OLED096-636, U10 LIS3DSHTR, U2 ATGM336H, U3 TPS62046DGQR, U4 HT-RA62, U5 Lever Switch TMHU26, U6 BQ24072RGT, U7 ESP32-S3-WROOM-1, U8 AT24C32A, U9 BME280

Commit message: Connect VSYS/3V3 sheet pins, sync R22, document remaining ERC state
Schematic/PCB edits: wire up the dangling VSYS and 3V3 hierarchical
sheet pins on the root sheet, and re-sync the board so R22 reads 1k
on both sides.

ERC 8 -> 6 errors; schematic parity 3 -> 2 issues; DRC still 0
violations and 0 unconnected pads.

README: explain each of the 6 remaining ERC errors (all PWR_FLAG /
no-connect annotations or the intentional JP3/JP4 jumper routing,
none of them wiring defects), and add an assembly note that JP3/JP4
ship unbridged and must be bridged for the display to receive power.

Co-Authored-By: Claude Opus 5 <noreply@anthropic.com>
Parts:
- R22: value 10k -> 1k

Commit message: Round board corners, re-annotate test points, rewrite README for GitHub
Board: 1.0 mm radius corners; outline now 71.00 x 46.00 mm.
Schematic: test points re-annotated to signal names (SDA1, SLC1,
CSN1, CLK1, MOSI1, MISO1, VS1, G1, G2, IO7, IO15, IO47, RST1, BOOT1).

README rewritten as a GitHub landing page: explains what the board is
for, adds Mermaid system-architecture and power-path diagrams, a
verified pin map traced from the netlist, board specs, and fab
instructions. Drops the ERC/DRC status and issue-tracking sections.

Co-Authored-By: Claude Opus 5 <noreply@anthropic.com>
Parts:
- added IO47: IO47, TestPoint:TestPoint_Pad_1.0x1.0mm, B.Cu at (113.0, 82.3)
- renumbered TP22 to 3V3, JP2 to BOOT1, TP15 to CLK, TP14 to CSN, TP26 to G, TP23 to G, TP19 to IO15, TP18 to IO7, TP17 to MISO, TP16 to MOSI, JP1 to RST1, TP12 to SDA, TP13 to SLC, TP21 to VS
Connections:
- U7 pad 24: unconnected-(U7-IO47-Pad24) -> /Microcontroller/IO47
Routing:
- net /Accelerometer/INT: track 29.4 -> 34.4 mm
- net /Microcontroller/IO47: track 0.00 -> 4.44 mm, vias 0 -> 1
Other:
- board size 71 x 46.1 mm -> 71 x 46 mm

Commit message: Add 3D renders and PCB layer views to README
- docs/meshtastic-v0-{f,b}.png: 3D renders of the populated board
- docs/layers-{front,back}.svg: F.Cu/B.Cu + silkscreen + outline plots
  exported with kicad-cli, back mirrored so silk reads correctly, on a
  dark canvas so they render in both GitHub themes
- README: hero render, side-by-side assembled and layer view galleries,
  and the kicad-cli commands to regenerate the plots
- Refresh board stats from kicad-cli pcb export stats: 90 footprints,
  342 pads (318 SMD / 22 TH), 71.0000 x 46.0000 mm

Co-Authored-By: Claude Opus 5 <noreply@anthropic.com>
Parts:
- added ?: LOGO, LOGO, F.Cu at (136.9, 104.5)
- added ?: LOGO, LOGO, F.Cu at (137.1, 104.5)
- renumbered BOOT1 to BOOT, RST1 to RST
Other:
- board text added: "8/2026"
- board text added: "by luthfai"
- board text added: "meshthingy_v0"
- board text removed: "meshtastic_thingy_v.0"
- board text removed: "xxxxxxxx"
