File: meshtastic-v0.kicad_sch (KiCad schematic)
At the start: 0 parts

Commit message: vib motor
Other:
- sheet Microcontroller ports: added VIB_MTR; removed none
- sheet Peripherals ports: added VIB_MTR; removed none
Changed lines of the file:
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@@
+	(wire
+		(pts
+			(xy 266.7 172.72) (xy 276.86 172.72)
+		)
+		(stroke
+			(width 0)
+			(type default)
+		)
+	)
 	(wire
 		(pts
@@
 			)
 		)
+		(pin "VIB_MTR" input
+			(at 276.86 172.72 180)
+			(effects
+				(font
+					(size 1.27 1.27)
+				)
+				(justify left)
+			)
+		)
 		(instances
 			(project "meshtastic-v0"
@@
 			(effects
 				(font
+					(size 1.27 1.27)
+				)
+				(justify right)
+			)
+		)
+		(pin "VIB_MTR" output
+			(at 266.7 172.72 0)
+			(effects
+				(font

Commit message: added vib motor fix
Other:
- sheet Microcontroller ports: added IO07; removed IO15, IO7
- sheet Peripherals ports: added IO07; removed IO15, IO7
Changed lines of the file:
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@@
-	(wire
-		(pts
-			(xy 266.7 193.04) (xy 276.86 193.04)
-		)
-		(stroke
-			(width 0)
-			(type default)
-		)
-	)
 	(wire
 		(pts
@@
 			)
 		)
-		(pin "IO15" bidirectional
-			(at 276.86 193.04 180)
-			(effects
-				(font
-					(size 1.27 1.27)
-				)
-				(justify left)
-			)
-		)
-		(pin "IO7" bidirectional
-			(at 276.86 190.5 180)
-			(effects
-				(font
-					(size 1.27 1.27)
-				)
-				(justify left)
-			)
-		)
 		(pin "STATUS_LED" input
 			(at 276.86 195.58 180)
@@
 		(pin "VIB_MTR" input
 			(at 276.86 172.72 180)
+			(effects
+				(font
+					(size 1.27 1.27)
+				)
+				(justify left)
+			)
+		)
+		(pin "IO07" bidirectional
+			(at 276.86 190.5 180)
 			(effects
 				(font
@@
 			)
 		)
-		(pin "IO7" bidirectional
-			(at 266.7 190.5 0)
-			(effects
-				(font
-					(size 1.27 1.27)
-				)
-				(justify right)
-			)
-		)
-		(pin "IO15" bidirectional
-			(at 266.7 193.04 0)
-			(effects
-				(font
-					(size 1.27 1.27)
-				)
-				(justify right)
-			)
-		)
 		(pin "IO47" bidirectional
 			(at 266.7 187.96 0)
@@
 			(effects
 				(font
+					(size 1.27 1.27)
+				)
+				(justify right)
+			)
+		)
+		(pin "IO07" bidirectional
+			(at 266.7 190.5 0)
+			(effects
+				(font
